Commit message: for new  model of gripper

File: src/mums_assistant/urdf/mums_assistant.urdf (robot description, URDF)
Before this commit: robot mums_assistant, 8 links, 7 joints
Links:
- link gripper_link_1: mass 0.0079633 -> 0.0096366
- link gripper_link_2: mass 0.0080391 -> 0.0096366
- link link_2: mass 0.064393 -> 0.064392
Joints:
- joint gripper_joint_1: axis -1 0 0 -> 0 0 -1; limit lower=-1.57 upper=1.57 effort=0.05 velocity=8.73 -> lower=-1.57 upper=0 effort=0.05 velocity=8.73; origin xyz=-0.0057476 0.004 0.037981 rpy=0 -0.0032835 0 -> xyz=0.003329 0.038 0.031999 rpy=-1.5708 1.569 -1.5707
- joint gripper_joint_2: axis -1 0 0 -> 0 0 1; mimic joint=gripper_joint_1 multiplier=-1 offset=0 -> joint=gripper_joint_1 multiplier=1 offset=0; origin xyz=-0.0058674 -0.023 0.037981 rpy=0 -0.0032835 0 -> xyz=0.0033427 0.038 0.0049991 rpy=-1.5708 1.5689 -1.5707
- joint joint_1: axis 0 0.16722 0.98592 -> 0 0 1; origin xyz=0 0 0.056 rpy=0.16801 0 0 -> xyz=0 0 0.056 rpy=0 0 0
- joint joint_2: axis 0 -1 0 -> 0 0 1; origin xyz=0.013919 0.006735 0.039709 rpy=-0.16801 0 0 -> xyz=0.013919 0 0.040276 rpy=1.5708 -0.4325 0
- joint joint_3: axis 0 1 0 -> 0 0 -1; origin xyz=0.0020606 0 0.11998 rpy=0 0.00077559 0 -> xyz=0 0.12 0 rpy=0 0 -0.41891
- joint joint_4: axis 1 0 0 -> 0.0013041 0.013594 0.99991; origin xyz=0.089732 0.0115 -0.0051 rpy=0.017845 0 0 -> xyz=0.089722 -0.0051 -0.0115 rpy=0 1.5695 -0.013594
- joint joint_5: axis 0 1 0 -> 0 0 1; origin xyz=0.028118 0 0.005 rpy=0 0 0 -> xyz=-0.0079737 0.0053658 0.027968 rpy=-1.4733 -1.5571 1.4752

Commit message: working gazebo and rviz connection

File: src/mums_assistant/urdf/mums_assistant.urdf (robot description, URDF)
Before this commit: robot mums_assistant, 8 links, 7 joints
Joints:
- joint gripper_joint_2: mimic joint=gripper_joint_1 multiplier=1 offset=0 -> joint=gripper_joint_1 multiplier=-1 offset=0

Commit message: added gripper_2 for control

File: src/mums_assistant/urdf/mums_assistant.urdf (robot description, URDF)
Before this commit: robot mums_assistant, 8 links, 7 joints
Joints:
- joint gripper_joint_2: limit lower=-1.57 upper=1.57 effort=0.05 velocity=8.73 -> lower=-1.57 upper=0 effort=0.05 velocity=8.73; mimic joint=gripper_joint_1 multiplier=-1 offset=0 -> (none); origin xyz=0.0033427 0.038 0.0049991 rpy=-1.5708 1.5689 -1.5707 -> xyz=0.0033427 0.038 0.0049991 rpy=-1.5707 1.5689 -1.5689

Commit message: gripper jitter fixed

File: src/mums_assistant/urdf/mums_assistant.urdf (robot description, URDF)
Before this commit: robot mums_assistant, 8 links, 7 joints
Links:
- link base_link: mass 0.096037 -> 10

Commit message: removed virtual_joint and added "world" link

File: src/mums_assistant/urdf/mums_assistant.urdf (robot description, URDF)
Before this commit: robot mums_assistant, 8 links, 7 joints
Links:
- added link world
Joints:
- added joint joint_0: type fixed, parent world, child base_link, origin xyz=0.0 0.0 0.0 rpy=0 0 0

Commit message: added models file and models in Rviz

File: src/mums_assistant/urdf/mums_assistant.urdf (robot description, URDF)
Before this commit: robot mums_assistant, 9 links, 8 joints
Links:
- added link mums_assistant_pedestal_link, mass 500; collision box size=0.15 0.15 0.5; visual box size=0.15 0.15 0.5
Joints:
- added joint ma_to_pedestal: type fixed, parent world, child base_link, origin xyz=0.0 0.0 0.5 rpy=0 0 0
- joint joint_0: child base_link -> mums_assistant_pedestal_link
